File: KCH.kicad_sch (KiCad schematic)
At the start: 15 parts, among them J1 CTBP9550/2, J2 Write EEPROM, J3 40HAT, J4 Serial, U1 CAT24C32WI

Commit message: Cleanup
Other:
- note added: "GPIO7 is used for boot 20% so that SPI CS function can be used to drive the pin from the device tree."
- note removed: "GPIOs for each LED can be swapped during layout Except GPIO7 is used for boot 20% so SPI CS function can be used to drive the pin from the device tree. PWM available on GPIO12/13"
Changed lines of the file:
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@@
   (title_block
     (title "KCH - Raspberry Pi HAT")
-    (date "2022-05-17")
-    (rev "S2")
+    (date "2022-06-28")
+    (rev "A (S2L1)")
     (company "Student Robotics")
   )
@@
     (stroke (width 0) (type default) (color 0 0 0 0))
   )
+  (text "Not populated as standard" (at 232.41 58.42 0)
+    (effects (font (size 1.27 1.27)) (justify left bottom))
+  )
   (text "40-Pin HAT Connector" (at 45.085 78.74 0)
     (effects (font (size 2.9972 2.9972) (thickness 0.5994) bold) (justify left bottom))
@@
     (effects (font (size 2.9972 2.9972) (thickness 0.5994) bold) (justify left bottom))
   )
-  (text "GPIOs for each LED can be swapped during layout\nExcept GPIO7 is used for boot 20% so SPI CS function \ncan be used to drive the pin from the device \ntree.\nPWM available on GPIO12/13"
+  (text "GPIO7 is used for boot 20% so that SPI CS function \ncan be used to drive the pin from the device \ntree."
     (at 203.835 90.805 0)
     (effects (font (size 1.27 1.27)) (justify left bottom))
