File: pcb/led.kicad_sch (KiCad schematic)
At the start: 45 parts, among them Q10 2N7002KDW, Q6 2N7002KDW, Q7 2N7002KDW, Q8 2N7002KDW, Q9 2N7002KDW

Commit message: Basic value changes
Parts:
- R21, R22, R28, R29, R31, R38, R43, R46: value 220R -> 3k3
- R32, R37: value 470R -> 1k
