File: pcb/rgb_led.kicad_sch (KiCad schematic)
At the start: 46 parts, among them Q11 2N7002KDW, Q12 2N7002KDW, Q13 2N7002KDW, Q14 2N7002KDW, Q15 2N7002KDW, Q16 2N7002KDW

Commit message: Basic value changes
Parts:
- R52, R61, R70, R79: value 330R -> 2k2
- R54, R63, R72, R81: value 220R -> 2k2
- R55, R64, R73, R82: value 220R -> 1k
