File: pcb/power.kicad_sch (KiCad schematic)
At the start: 43 parts, among them Q1 AO3407A, Q2 PMV20EN, Q3 NCE3401AY, Q4 NCE3401AY, Q5 DMMT5401, U2 AP3200T

Commit message: Correct regulator name
Parts:
- U2: value AP3200T -> AP63200T
Changed lines of the file:
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@@
   (title_block
     (title "KCH - Raspberry Pi HAT")
-    (date "2022-07-15")
+    (date "2022-07-16")
     (rev "B (S3L2)")
     (company "Student Robotics")
@@
     (in_bom yes) (on_board yes) (fields_autoplaced)
     (property "Reference" "U2" (id 0) (at 111.76 55.88 0))
-    (property "Value" "AP3200T" (id 1) (at 111.76 58.42 0))
+    (property "Value" "AP63200T" (id 1) (at 111.76 58.42 0))
     (property "Footprint" "Package_TO_SOT_SMD:SOT-23-6" (id 2) (at 111.76 58.42 0)
       (effects (font (size 1.27 1.27)) hide)
